File: torpedy/torpedy.kicad_pcb (KiCad board)
At the start: 2 copper layers, 63.5 x 107.9 mm, 41 parts, among them J1 RPi I/O, J2 V_IN+, J3 V_IN-, J4 Zasilanie Serwa, J5 Batt HP, J6 Torpedo, J7 Torpedo EM, J8 V_OUT+, J9 V_OUT-, Q1 Q_NPN_BEC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

Commit message: Schemat pcb - początek
Parts:
- R14, R15, R16, R8: moved to F.Cu
- moved J7 143.9 mm to (178.4, 135.9), turned to 0 degrees
- moved J4 129.9 mm to (182.9, 47.0)
- moved D2 126.9 mm to (170.8, 133.3), turned to 90 degrees
- moved Q4 119.9 mm to (179.7, 116.8), turned to 270 degrees
- moved J5 116.7 mm to (196.8, 41.9), turned to 0 degrees
- moved R8 116.1 mm to (200.7, 78.7)
- moved R16 111.9 mm to (221.0, 71.1)
- moved R15 109.6 mm to (221.0, 63.5)
- moved R14 109.4 mm to (200.7, 55.9)
- moved J6 109.1 mm to (170.2, 39.4)
- moved R13 108.1 mm to (181.2, 105.4), turned to 0 degrees
- moved J2 105.4 mm to (177.8, 73.7), turned to 180 degrees
- moved D3 104.4 mm to (170.8, 114.3), turned to 90 degrees
- moved Q3 104.1 mm to (181.3, 96.3), turned to 90 degrees
- moved R11 101.7 mm to (181.2, 102.2), turned to 180 degrees
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Connections:
- J1 pad 4: Trigger -> Charger_R.C.
- J1 pad 5: Charger_R.C. -> Trigger
Routing:
- net Cewka+: track 0.00 -> 127.0 mm
- net Net-(Q3-Pad3): track 0.00 -> 18.9 mm
- net Net-(Q3-Pad1): track 0.00 -> 16.5 mm
- net Net-(Q3-Pad2): track 0.00 -> 13.3 mm
- net reed_switch: track 0.00 -> 3.88 mm
- net Net-(R10-Pad1): track 0.00 -> 3.81 mm
- added copper zone on F.Cu, net Cewka-
Other:
- board size 63.5 x 107.9 mm -> 63.5 x 110.5 mm

Commit message: wersja finalna
Parts:
- removed R15, R16: 150, Resistor_THT:R_Axial_DIN0414_L11.9mm_D4.5mm_P20.32mm_Horizontal
- R14, R8: value 150 -> 300; moved to B.Cu
- moved R14 140.2 mm to (75.4, 118.9)
- moved R8 129.7 mm to (75.4, 112.6)
- moved J5 122.2 mm to (82.5, 85.1), turned to 180 degrees
- moved J9 119.4 mm to (62.1, 106.7), turned to 0 degrees
- moved J8 118.7 mm to (70.5, 106.7), turned to 0 degrees
- moved J3 108.1 mm to (62.1, 75.7), turned to 0 degrees
- moved J2 107.3 mm to (70.5, 75.7), turned to 0 degrees
- moved R10 99.4 mm to (76.2, 61.2), turned to 90 degrees
- moved U4 98.0 mm to (84.1, 63.5)
- moved R12 91.0 mm to (94.9, 59.4)
- moved C6 90.7 mm to (73.7, 134.0), turned to 90 degrees
- moved Q3 90.3 mm to (97.6, 62.5), turned to 180 degrees
- moved C5 88.2 mm to (73.7, 147.3), turned to 270 degrees
- moved R11 87.8 mm to (102.9, 62.6), turned to 270 degrees
- moved R13 87.1 mm to (105.4, 62.6), turned to 90 degrees
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Connections:
- J1 pad 1: +3V3 -> GNDD
- J1 pad 2: RPi_reed_switch -> +3V3
- J1 pad 3: RPi_serwo_pwm -> Charger_R.C.
- J1 pad 4: Charger_R.C. -> Trigger
- J1 pad 5: Trigger -> RPi_reed_switch
- J1 pad 6: GNDD -> RPi_serwo_pwm
- J6 pad 1: -BATT -> PWM_serwo
- J6 pad 4: PWM_serwo -> -BATT
- J8 pad 1: +BATT -> Net-(J8-Pad1)
- R14 pad 1: +BATT -> Net-(J8-Pad1)
- R14 pad 2: Net-(R14-Pad2) -> Cewka+
- R8 pad 1: +BATT -> Net-(J8-Pad1)
- R8 pad 2: Net-(R16-Pad1) -> Cewka+
Routing:
- net +BATT: track 0.00 -> 145.8 mm, vias 0 -> 2
- net -BATT: track 0.00 -> 138.8 mm, vias 0 -> 6
- net Cewka+: track 127.0 -> 47.7 mm
- net Net-(Q1-Pad2): track 0.00 -> 75.9 mm
- net reed_switch: track 3.88 -> 27.2 mm
- net Net-(Q3-Pad2): track 13.3 -> 36.0 mm
- net RPi_reed_switch: track 0.00 -> 22.5 mm
- net PWM_serwo: track 0.00 -> 21.6 mm
- net Charger_R.C.: track 0.00 -> 19.2 mm
- net Trigger: track 0.00 -> 15.7 mm
- net Net-(Q1-Pad1): track 0.00 -> 14.6 mm
- net Net-(J8-Pad1): track 0.00 -> 14.3 mm
- net Net-(J3-Pad1): track 0.00 -> 12.8 mm
- net RPi_serwo_pwm: track 0.00 -> 11.8 mm
- net V+_serwo: track 0.00 -> 8.44 mm
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- added copper zone on F.Cu, net Cewka+
- added copper zone on F.Cu, net GNDD
Other:
- board size 63.5 x 110.5 mm -> 63.5 x 116.8 mm
