File: torpedy/torpedy.sch (KiCad schematic (older format))
At the start: 46 parts

Commit message: kilka poprawek wartości elementow
Parts:
- removed D?: TVS_18V, symbol Device:D_TVS
- added D1: 18V, symbol Device:D_Zener
- C1, C2, C3, C4, C5, C6: renamed from C?; footprint (none) -> Capacitor_THT:CP_Radial_D16.0mm_P7.50mm
- D3: renamed from D?; value TVS_18V -> TVS_30V
- gave numbers to parts that had none: 38
Other:
- note added: "C: \nSrednica: >16mm\nwysokosc: >36mm\nrozstaw: <8mm"
- note added: "MAX 30V"

Commit message: poprawki parametrów elementów
Parts:
- removed C4: 2200u, Capacitor_THT:CP_Radial_D16.0mm_P7.50mm, symbol Device:CP
- added C7: 2200u, Capacitor_THT:CP_Radial_D16.0mm_P7.50mm, symbol Device:CP
- D3: value TVS_30V -> TVS_24V
- Q2, Q4: value N_MOS -> IRL2203N
Connections:
- wire segments 140 -> 138
Other:
- moved on the sheet: C1, C2, C3, C5, C6
Changed lines of the file:
@@
 encoding utf-8
 Sheet 1 1
-Title ""
-Date ""
-Rev ""
-Comp ""
+Title "Układ zasilania wyrzutni torped"
+Date "2019-07-16"
+Rev "1"
+Comp "KN Robocik"
 Comment1 ""
 Comment2 ""
@@
 P 10450 3750
 F 0 "Q4" V 10350 3800 50  0000 L CNN
-F 1 "N_MOS" V 10700 3650 50  0000 L CNN
+F 1 "IRL2203N" V 10700 3650 50  0000 L CNN
 F 2 "" H 10650 3850 50  0001 C CNN
 F 3 "~" H 10450 3750 50  0001 C CNN
@@
 Text GLabel 10550 2950 1    50   Input ~ 0
 PowerBank
-Text GLabel 6950 3100 2    50   Input ~ 0
+Text GLabel 6600 3250 2    50   Input ~ 0
 PowerBank
 $Comp
@@
 P 10900 3700
 F 0 "D3" H 10850 3600 50  0000 L CNN
-F 1 "TVS_30V" H 10750 3800 50  0000 L CNN
+F 1 "TVS_24V" H 10750 3800 50  0000 L CNN
 F 2 "" H 10900 3700 50  0001 C CNN
 F 3 "~" H 10900 3700 50  0001 C CNN
@@
 L Device:CP C6
 U 1 1 5D2E6268
-P 7400 3450
-F 0 "C6" V 7250 3400 50  0000 L CNN
-F 1 "2200u" V 7550 3350 50  0000 L CNN
-F 2 "Capacitor_THT:CP_Radial_D16.0mm_P7.50mm" H 7438 3300 50  0001 C CNN
-F 3 "~" H 7400 3450 50  0001 C CNN
-	1    7400 3450
-	1    0    0    -1
+P 5650 3050
+F 0 "C6" V 5500 3000 50  0000 L CNN
+F 1 "2200u" V 5800 2950 50  0000 L CNN
+F 2 "Capacitor_THT:CP_Radial_D16.0mm_P7.50mm" H 5688 2900 50  0001 C CNN
+F 3 "~" H 5650 3050 50  0001 C CNN
+	1    5650 3050
+	-1   0    0    1
 $EndComp
 $Comp
 L Device:CP C5
 U 1 1 5D2E6386
-P 7000 3450
-F 0 "C5" V 6850 3400 50  0000 L CNN
-F 1 "2200u" V 7150 3350 50  0000 L CNN
-F 2 "Capacitor_THT:CP_Radial_D16.0mm_P7.50mm" H 7038 3300 50  0001 C CNN
-F 3 "~" H 7000 3450 50  0001 C CNN
-	1    7000 3450
-	1    0    0    -1
-$EndComp
-$Comp
-L Device:CP C4
-U 1 1 5D2E648C
-P 6600 3450
-F 0 "C4" V 6450 3400 50  0000 L CNN
-F 1 "2200u" V 6750 3350 50  0000 L CNN
-F 2 "Capacitor_THT:CP_Radial_D16.0mm_P7.50mm" H 6638 3300 50  0001 C CNN
-F 3 "~" H 6600 3450 50  0001 C CNN
-	1    6600 3450
-	1    0    0    -1
+P 6050 3050
+F 0 "C5" V 5900 3000 50  0000 L CNN
+F 1 "2200u" V 6200 2950 50  0000 L CNN
+F 2 "Capacitor_THT:CP_Radial_D16.0mm_P7.50mm" H 6088 2900 50  0001 C CNN
+F 3 "~" H 6050 3050 50  0001 C CNN
+	1    6050 3050
+	-1   0    0    1
 $EndComp
 $Comp
 L Device:CP C3
 U 1 1 5D2E64D4
-P 6200 3450
-F 0 "C3" V 6050 3400 50  0000 L CNN
-F 1 "2200u" V 6350 3350 50  0000 L CNN
-F 2 "Capacitor_THT:CP_Radial_D16.0mm_P7.50mm" H 6238 3300 50  0001 C CNN
-F 3 "~" H 6200 3450 50  0001 C CNN
-	1    6200 3450
-	1    0    0    -1
-$EndComp
-Wire Wire Line
-	6200 3250 6200 3300
+P 6450 3450
+F 0 "C3" V 6300 3400 50  0000 L CNN
+F 1 "2200u" V 6600 3350 50  0000 L CNN
+F 2 "Capacitor_THT:CP_Radial_D16.0mm_P7.50mm" H 6488 3300 50  0001 C CNN
+F 3 "~" H 6450 3450 50  0001 C CNN
+	1    6450 3450
+	1    0    0    -1
+$EndComp
 $Comp
 L power:GNDA #PWR0103
 U 1 1 5D2E7DE1
-P 6200 3750
-F 0 "#PWR0103" H 6200 3500 50  0001 C CNN
-F 1 "GNDA" H 6205 3577 50  0000 C CNN
-F 2 "" H 6200 3750 50  0001 C CNN
-F 3 "" H 6200 3750 50  0001 C CNN
-	1    6200 3750
-	1    0    0    -1
-$EndComp
-Wire Wire Line
-	6200 3650 6200 3600
-Wire Wire Line
-	6200 3750 6200 3650
-Connection ~ 6200 3650
+P 6250 3750
+F 0 "#PWR0103" H 6250 3500 50  0001 C CNN
+F 1 "GNDA" H 6255 3577 50  0000 C CNN
+F 2 "" H 6250 3750 50  0001 C CNN
+F 3 "" H 6250 3750 50  0001 C CNN
+	1    6250 3750
+	1    0    0    -1
+$EndComp
 $Comp
 L Device:R R8
@@
 	0    -1   -1   0
 $EndComp
-Text Notes 5100 3000 0    50   ~ 0
+Text Notes 4800 3150 1    50   ~ 0
 30V - 300mA ??
 $Comp
@@
 Wire Wire Line
 	4500 3350 4900 3350
-Wire Wire Line
-	4900 3350 4900 3650
 $Comp
 L power:VCC #PWR0104
@@
 P 2800 3650
 F 0 "Q2" V 2700 3700 50  0000 L CNN
-F 1 "N_MOS" V 3050 3550 50  0000 L CNN
+F 1 "IRL2203N" V 3050 3550 50  0000 L CNN
 F 2 "" H 3000 3750 50  0001 C CNN
 F 3 "~" H 2800 3650 50  0001 C CNN
@@
 L Device:CP C2
 U 1 1 5D44DEA8
-P 5800 3450
-F 0 "C2" V 5650 3400 50  0000 L CNN
-F 1 "2200u" V 5950 3350 50  0000 L CNN
-F 2 "Capacitor_THT:CP_Radial_D16.0mm_P7.50mm" H 5838 3300 50  0001 C CNN
-F 3 "~" H 5800 3450 50  0001 C CNN
-	1    5800 3450
+P 6050 3450
+F 0 "C2" V 5900 3400 50  0000 L CNN
+F 1 "2200u" V 6200 3350 50  0000 L CNN
+F 2 "Capacitor_THT:CP_Radial_D16.0mm_P7.50mm" H 6088 3300 50  0001 C CNN
+F 3 "~" H 6050 3450 50  0001 C CNN
+	1    6050 3450
 	1    0    0    -1
 $EndComp
@@
 L Device:CP C1
 U 1 1 5D44DF18
-P 5400 3450
-F 0 "C1" V 5250 3400 50  0000 L CNN
-F 1 "2200u" V 5550 3350 50  0000 L CNN
-F 2 "Capacitor_THT:CP_Radial_D16.0mm_P7.50mm" H 5438 3300 50  0001 C CNN
-F 3 "~" H 5400 3450 50  0001 C CNN
-	1    5400 3450
-	1    0    0    -1
-$EndComp
-Wire Wire Line
-	5800 3300 5800 3250
-Connection ~ 5800 3250
-Wire Wire Line
-	5800 3250 6200 3250
-Wire Wire Line
-	5400 3300 5400 3250
-Wire Wire Line
-	5400 3250 5800 3250
-Wire Wire Line
-	5400 3600 5400 3650
-Wire Wire Line
-	5400 3650 5800 3650
-Wire Wire Line
-	5800 3600 5800 3650
-Connection ~ 5800 3650
-Wire Wire Line
-	5800 3650 6200 3650
+P 5650 3450
+F 0 "C1" V 5500 3400 50  0000 L CNN
+F 1 "2200u" V 5800 3350 50  0000 L CNN
+F 2 "Capacitor_THT:CP_Radial_D16.0mm_P7.50mm" H 5688 3300 50  0001 C CNN
+F 3 "~" H 5650 3450 50  0001 C CNN
+	1    5650 3450
+	1    0    0    -1
+$EndComp
 $Comp
 L Isolator:LTV-817 U3
@@
 Text Notes 7950 700  0    59   ~ 12
 Przyłącze przewodu od torped
-Connection ~ 6200 3250
-Wire Wire Line
-	7400 3600 7400 3650
-Wire Wire Line
-	7400 3650 7000 3650
-Connection ~ 7000 3650
-Wire Wire Line
-	7000 3600 7000 3650
-Wire Wire Line
-	7000 3650 6600 3650
-Wire Wire Line
-	6600 3650 6200 3650
-Connection ~ 6600 3650
-Wire Wire Line
-	6600 3600 6600 3650
-Wire Wire Line
-	7400 3300 7400 3250
-Wire Wire Line
-	7400 3250 7000 3250
-Connection ~ 7000 3250
-Wire Wire Line
-	7000 3300 7000 3250
-Wire Wire Line
-	7000 3250 6600 3250
-Wire Wire Line
-	6600 3250 6200 3250
-Connection ~ 6600 3250
-Wire Wire Line
-	6600 3300 6600 3250
-Wire Wire Line
-	5400 3650 4900 3650
-Connection ~ 5400 3650
-Wire Wire Line
-	5300 3250 5400 3250
-Connection ~ 5400 3250
 Wire Wire Line
 	9850 3750 10150 3750
@@
 	10150 4150 9850 4150
 Connection ~ 10150 4150
-Wire Wire Line
-	6950 3100 6600 3100
-Wire Wire Line
-	6600 3100 6600 3250
 Wire Notes Line
 	7850 2200 7850 4550
@@
 	0    1    1    0
 $EndComp
-Text Notes 6000 2750 0    79   ~ 16
+Text Notes 5650 2750 0    79   ~ 16
 C: \nSrednica: >16mm\nwysokosc: >36mm\nrozstaw: <8mm
+$Comp
+L Device:CP C7
+U 1 1 5D761C77
+P 6450 3050
+F 0 "C7" V 6300 3000 50  0000 L CNN
+F 1 "2200u" V 6600 2950 50  0000 L CNN
+F 2 "Capacitor_THT:CP_Radial_D16.0mm_P7.50mm" H 6488 2900 50  0001 C CNN
+F 3 "~" H 6450 3050 50  0001 C CNN
+	1    6450 3050
+	-1   0    0    1
+$EndComp
+Wire Wire Line
+	5650 3600 5650 3700
+Wire Wire Line
+	5650 3700 6050 3700
+Wire Wire Line
+	6250 3750 6250 3700
+Connection ~ 6250 3700
+Wire Wire Line
+	6250 3700 6450 3700
+Wire Wire Line
+	6450 3600 6450 3700
+Wire Wire Line
+	6050 3600 6050 3700
+Connection ~ 6050 3700
+Wire Wire Line
+	6050 3700 6250 3700
+Wire Wire Line
+	6450 3200 6450 3250
+Connection ~ 6450 3250
+Wire Wire Line
+	6450 3300 6450 3250
+Wire Wire Line
+	6050 3300 6050 3250
+Connection ~ 6050 3250
+Wire Wire Line
+	6050 3250 6450 3250
+Wire Wire Line
+	6050 3250 6050 3200
+Wire Wire Line
+	5650 3200 5650 3250
+Connection ~ 5650 3250
+Wire Wire Line
+	5650 3250 6050 3250
+Wire Wire Line
+	5650 3250 5650 3300
+Wire Wire Line
+	4900 3350 4900 3700
+Connection ~ 5650 3700
+Wire Wire Line
+	5650 2900 5650 2850
+Wire Wire Line
+	5650 2850 6050 2850
+Wire Wire Line
+	6450 2900 6450 2850
+Connection ~ 6450 2850
+Wire Wire Line
+	6050 2900 6050 2850
+Connection ~ 6050 2850
+Wire Wire Line
+	6050 2850 6450 2850
+$Comp
+L power:GNDA #PWR01
+U 1 1 5D7F7A14
+P 6800 2900
+F 0 "#PWR01" H 6800 2650 50  0001 C CNN
+F 1 "GNDA" H 6805 2727 50  0000 C CNN
+F 2 "" H 6800 2900 50  0001 C CNN
+F 3 "" H 6800 2900 50  0001 C CNN
+	1    6800 2900
+	1    0    0    -1
+$EndComp
+Wire Wire Line
+	6800 2900 6800 2850
+Wire Wire Line
+	6450 3250 6600 3250
+Wire Wire Line
+	6450 2850 6800 2850
+Wire Wire Line
+	5300 3250 5650 3250
+Wire Wire Line
+	4900 3700 5650 3700
 $EndSCHEMATC

Commit message: Poprawki schematu
Parts:
- removed D1: 18V, symbol Device:D_Zener
- J1: value Enable -> Charger R.C.
- J5: value Vbatt - zasilanie cewki -> Batt HP
- J6: value sygnały_rpi -> RPi I/O
Connections:
- net labels added: +BATT, -BATT
- net labels removed: GNDA, VCC, VDD, gndd
- wire segments 138 -> 128
Other:
- moved on the sheet: D2, D3, J5, J6, Q4, R13, R3, R6, R7, R9, U3

Commit message: Jprdl nic nie umie i gupi jeste
Parts:
- removed J1: Charger R.C., symbol Connector_Generic:Conn_01x02
- removed J10: żółty, symbol Connector_Generic:Conn_01x01
- removed J11: zielony, symbol Connector_Generic:Conn_01x01
- removed J12: różowy, symbol Connector_Generic:Conn_01x01
- removed J13: niebieski, symbol Connector_Generic:Conn_01x01
- removed J14: czerwony, symbol Connector_Generic:Conn_01x01
- removed J15: brązowy, symbol Connector_Generic:Conn_01x01
- removed J16: ekran, symbol Connector_Generic:Conn_01x01
- removed J2: step_up - Vin, symbol Connector_Generic:Conn_01x02
- removed J3: step_up - Vout, symbol Connector_Generic:Conn_01x02
- removed Q1, Q3: Q_NPN_BCE, symbol Device:Q_NPN_BCE
- added J1: RPi I/O, Connector_Molex:Molex_SPOX_5267-06A_1x06_P2.50mm_Vertical, symbol Connector_Generic:Conn_01x06
- added J2: V_IN+, Connector_PinHeader_2.54mm:PinHeader_1x01_P2.54mm_Vertical, symbol Connector_Generic:Conn_01x01
- added J3: V_IN-, Connector_PinHeader_2.54mm:PinHeader_1x01_P2.54mm_Vertical, symbol Connector_Generic:Conn_01x01
- added Q1, Q3: Q_NPN_BEC, Package_TO_SOT_SMD:SOT-23_Handsoldering, symbol Device:Q_NPN_BEC
- added R14, R15, R16: 150, Resistor_THT:R_Axial_DIN0414_L11.9mm_D4.5mm_P20.32mm_Horizontal, symbol Device:R
- D2: footprint (none) -> Diode_SMD:D_SMC_Handsoldering
- D3: footprint (none) -> Diode_SMD:D_SMB_Handsoldering
- J4, J5: footprint (none) -> Connector_Molex:Molex_Mini-Fit_Jr_5566-02A_2x01_P4.20mm_Vertical
- J6: value RPi I/O -> Torpedo; footprint (none) -> Connector_Molex:Molex_SPOX_5267-04A_1x04_P2.50mm_Vertical
- J7: value Trigger -> Torpedo EM; footprint (none) -> Connector_Molex:Molex_Mini-Fit_Jr_5566-02A_2x01_P4.20mm_Vertical
- J8: value biały -> V_OUT+; footprint (none) -> Connector_PinHeader_2.54mm:PinHeader_1x01_P2.54mm_Vertical
- J9: value szary -> V_OUT-; footprint (none) -> Connector_PinHeader_2.54mm:PinHeader_1x01_P2.54mm_Vertical
- Q2, Q4: footprint (none) -> Package_TO_SOT_SMD:TO-263-2
- R1, R10, R11, R12, R13, R2, R3, R4, R5, R6, R7, R9: footprint (none) -> Resistor_SMD:R_0805_2012Metric_Pad1.15x1.40mm_HandSolder
- R8: value 100 -> 150; footprint (none) -> Resistor_THT:R_Axial_DIN0414_L11.9mm_D4.5mm_P20.32mm_Horizontal
- U1, U2, U3, U4: footprint Package_DIP:DIP-4_W7.62mm -> Package_DIP:SMDIP-4_W9.53mm
Connections:
- net +3V3: now also J1.1 (Pin_1); no longer J6.1 (Pin_1)
- net +BATT: now also J8.1 (Pin_1), J2.1 (Pin_1), R14.1
- net -BATT: now also J6.1 (Pin_1), J9.1 (Pin_1); no longer J8.1 (Pin_1)
- net Cewka+: now also J7.1 (Pin_1), R15.2, R16.2; no longer R8.2
- net Cewka-: now also J7.2 (Pin_2)
- net GNDD: now also U1.2, U4.2, J1.6 (Pin_6); no longer J6.4 (Pin_4)
- net PWM_serwo: now also J6.4 (Pin_4)
- net RPi_reed_switch: now also J1.2 (Pin_2); no longer J6.2 (Pin_2)
- net RPi_serwo_pwm: now also J1.3 (Pin_3); no longer J6.3 (Pin_3)
- net V+_serwo: now also J6.3 (Pin_3)
- net reed_switch: now also J6.2 (Pin_2); no longer J9.1 (Pin_1)
- net at Q4.1 (G), R11.1, R13.2: now also Q3.2 (E)
- net at R12.1, U4.4: now also Q3.3 (C)
- net at R11.2, U4.3: now also Q3.1 (B)
- net Trigger: now reaches R10.2
- net Trigger: now also J1.4 (Pin_4); no longer J7.1 (Pin_1)
- net at Q2.2 (D): now also J3.1 (Pin_1)
- net at Q2.1 (G), R2.1, R5.2: now also Q1.2 (E)
- net at R4.1, U1.4: now also Q1.3 (C)
- net at R2.2, U1.3: now also Q1.1 (B)
- net Charger_R.C.: now reaches R1.2
- net Charger_R.C.: now also J1.5 (Pin_5)
- new net: R16.1, R8.2
- new net: R14.2, R15.1
Other:
- note added: "27V - 300mA ??"
- note added: "MAX 27V"
- note removed: "30V - 300mA ??"
- note removed: "MAX 30V"
- moved on the sheet: C1, C2, C3, C5, C6, C7, Q2, R1, R2, R4, R5, R8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

Commit message: Schemat pcb - początek
Connections:
- net Charger_R.C.: now also J1.4 (Pin_4); no longer J1.5 (Pin_5)
- net Trigger: now also J1.5 (Pin_5); no longer J1.4 (Pin_4)
Changed lines of the file:
@@
 EESchema Schematic File Version 4
 LIBS:torpedy-cache
-EELAYER 29 0
+EELAYER 26 0
 EELAYER END
 $Descr A4 11693 8268
@@
 Text GLabel 8500 3250 0    59   Input ~ 0
 Trigger
+Text GLabel 6950 1550 2    39   Output ~ 0
+Trigger
 Text GLabel 6950 1450 2    39   Output ~ 0
-Trigger
-Text GLabel 6950 1550 2    39   Output ~ 0
 Charger_R.C.
 $Comp

Commit message: wersja finalna
Parts:
- removed R15, R16: 150, Resistor_THT:R_Axial_DIN0414_L11.9mm_D4.5mm_P20.32mm_Horizontal, symbol Device:R
- R14, R8: value 150 -> 300
Connections:
- net +3V3: now also J1.2 (Pin_2); no longer J1.1 (Pin_1)
- net +BATT: no longer J8.1 (Pin_1), R14.1, R8.1
- net -BATT: now also J6.4 (Pin_4); no longer J6.1 (Pin_1)
- net Cewka+: now also R14.2, R8.2
- net Charger_R.C.: now also J1.3 (Pin_3); no longer J1.4 (Pin_4)
- net GNDD: now also J1.1 (Pin_1); no longer J1.6 (Pin_6)
- net PWM_serwo: now also J6.1 (Pin_1); no longer J6.4 (Pin_4)
- net RPi_reed_switch: now also J1.5 (Pin_5); no longer J1.2 (Pin_2)
- net RPi_serwo_pwm: now also J1.6 (Pin_6); no longer J1.3 (Pin_3)
- net Trigger: now also J1.4 (Pin_4); no longer J1.5 (Pin_5)
- new net: J8.1 (Pin_1), R14.1, R8.1
Changed lines of the file:
@@
 P 5500 3300
 F 0 "R8" V 5385 3300 50  0000 C CNN
-F 1 "150" V 5294 3300 50  0000 C CNN
+F 1 "300" V 5294 3300 50  0000 C CNN
 F 2 "Resistor_THT:R_Axial_DIN0414_L11.9mm_D4.5mm_P20.32mm_Horizontal" V 5430 3300 50  0001 C CNN
 F 3 "~" H 5500 3300 50  0001 C CNN
@@
 Text Notes 4800 2950 2    50   ~ 0
 27V - 300mA ??
-Wire Wire Line
-	5250 2750 5250 3050
 Wire Wire Line
 	5250 3300 5350 3300
@@
 Text GLabel 9950 1450 0    39   Input ~ 0
 Cewka-
-Text GLabel 9000 1600 0    39   Input ~ 0
+Text GLabel 9000 1300 0    39   Input ~ 0
 PWM_serwo
 Text GLabel 9000 1500 0    39   Input ~ 0
 V+_serwo
-Text GLabel 9000 1300 0    39   Input ~ 0
+Text GLabel 9000 1600 0    39   Input ~ 0
 -BATT
 Text GLabel 9000 1400 0    39   Output ~ 0
@@
 $EndComp
 $Comp
-L power:+BATT #PWR0105
-U 1 1 5D2FBF16
-P 5250 2750
-F 0 "#PWR0105" H 5250 2600 50  0001 C CNN
-F 1 "+BATT" H 5265 2923 50  0000 C CNN
-F 2 "" H 5250 2750 50  0001 C CNN
-F 3 "" H 5250 2750 50  0001 C CNN
-	1    5250 2750
-	1    0    0    -1
-$EndComp
-$Comp
 L power:-BATT #PWR0106
 U 1 1 5D2FC313
@@
 Connection ~ 4950 1450
 Wire Wire Line
+	6950 1450 6850 1450
+Wire Wire Line
 	6950 1350 6850 1350
-Wire Wire Line
-	6950 1250 6850 1250
 Wire Wire Line
 	4900 1350 5100 1350
@@
 	-1   0    0    1
 $EndComp
-Text GLabel 6950 1250 2    39   Input ~ 0
+Text GLabel 6950 1550 2    39   Input ~ 0
 RPi_reed_switch
 $Comp
@@
 	1    0    0    -1
 $EndComp
-Text GLabel 6950 1350 2    39   Output ~ 0
+Text GLabel 6950 1650 2    39   Output ~ 0
 RPi_serwo_pwm
 $Comp
 L power:GNDD #PWR0118
 U 1 1 5D540B85
-P 7050 1700
-F 0 "#PWR0118" H 7050 1450 50  0001 C CNN
-F 1 "GNDD" H 7054 1545 50  0000 C CNN
-F 2 "" H 7050 1700 50  0001 C CNN
-F 3 "" H 7050 1700 50  0001 C CNN
-	1    7050 1700
-	-1   0    0    -1
-$EndComp
-Wire Wire Line
-	7050 1150 7050 1100
-Wire Wire Line
-	6850 1150 7050 1150
-$Comp
-L power:+3V3 #PWR0117
-U 1 1 5D53B98C
 P 7050 1100
-F 0 "#PWR0117" H 7050 950 50  0001 C CNN
-F 1 "+3V3" H 7065 1273 50  0000 C CNN
+F 0 "#PWR0118" H 7050 850 50  0001 C CNN
+F 1 "GNDD" H 7054 945 50  0000 C CNN
 F 2 "" H 7050 1100 50  0001 C CNN
 F 3 "" H 7050 1100 50  0001 C CNN
 	1    7050 1100
+	1    0    0    1
+$EndComp
+Wire Wire Line
+	6850 1150 7050 1150
+$Comp
+L power:+3V3 #PWR0117
+U 1 1 5D53B98C
+P 7300 1100
+F 0 "#PWR0117" H 7300 950 50  0001 C CNN
+F 1 "+3V3" H 7315 1273 50  0000 C CNN
+F 2 "" H 7300 1100 50  0001 C CNN
+F 3 "" H 7300 1100 50  0001 C CNN
+	1    7300 1100
 	-1   0    0    -1
 $EndComp
@@
 Text GLabel 8500 3250 0    59   Input ~ 0
 Trigger
-Text GLabel 6950 1550 2    39   Output ~ 0
+Text GLabel 6950 1450 2    39   Output ~ 0
 Trigger
-Text GLabel 6950 1450 2    39   Output ~ 0
+Text GLabel 6950 1350 2    39   Output ~ 0
 Charger_R.C.
 $Comp
@@
 $EndComp
 Wire Wire Line
-	7050 1700 7050 1650
-Wire Wire Line
-	7050 1650 6850 1650
-Wire Wire Line
-	6950 1550 6850 1550
-Wire Wire Line
-	6850 1450 6950 1450
+	6950 1650 6850 1650
+Wire Wire Line
+	6850 1550 6950 1550
 $Comp
 L Connector_Generic:Conn_01x04 J6
@@
 P 5500 3050
 F 0 "R14" V 5707 3050 50  0000 C CNN
-F 1 "150" V 5616 3050 50  0000 C CNN
+F 1 "300" V 5616 3050 50  0000 C CNN
 F 2 "Resistor_THT:R_Axial_DIN0414_L11.9mm_D4.5mm_P20.32mm_Horizontal" V 5430 3050 50  0001 C CNN
 F 3 "~" H 5500 3050 50  0001 C CNN
@@
 Wire Wire Line
 	5350 3050 5250 3050
-Connection ~ 5250 3050
 Wire Wire Line
 	5250 3050 5250 3200
 Wire Wire Line
-	6050 3300 6100 3300
-$Comp
-L Device:R R16
-U 1 1 5D5DBF1F
-P 5900 3300
-F 0 "R16" V 5785 3300 50  0000 C CNN
-F 1 "150" V 5694 3300 50  0000 C CNN
-F 2 "Resistor_THT:R_Axial_DIN0414_L11.9mm_D4.5mm_P20.32mm_Horizontal" V 5830 3300 50  0001 C CNN
-F 3 "~" H 5900 3300 50  0001 C CNN
-	1    5900 3300
-	0    -1   -1   0
-$EndComp
-$Comp
-L Device:R R15
-U 1 1 5D5DBD8D
-P 5900 3050
-F 0 "R15" V 6107 3050 50  0000 C CNN
-F 1 "150" V 6016 3050 50  0000 C CNN
-F 2 "Resistor_THT:R_Axial_DIN0414_L11.9mm_D4.5mm_P20.32mm_Horizontal" V 5830 3050 50  0001 C CNN
-F 3 "~" H 5900 3050 50  0001 C CNN
-	1    5900 3050
-	0    -1   -1   0
-$EndComp
-Wire Wire Line
 	6100 3300 6100 3050
-Wire Wire Line
-	6100 3050 6050 3050
 Connection ~ 6100 3300
 Wire Wire Line
 	6100 3300 6350 3300
 Wire Wire Line
-	5650 3300 5750 3300
-Wire Wire Line
-	5650 3050 5750 3050
+	7050 1150 7050 1100
+Wire Wire Line
+	7300 1100 7300 1250
+Wire Wire Line
+	7300 1250 6850 1250
+Wire Wire Line
+	5650 3050 6100 3050
+Wire Wire Line
+	5650 3300 6100 3300
 $EndSCHEMATC
